File: pcb/pcb_module_hx711/pcb_module_hx711.kicad_pcb (KiCad board)
At the start: 2 copper layers, 106.4 x 81.5 mm, 89 parts, among them J1 E+, J2 E-, J3 S+, J4 S-, J5 RFShield_TwoPieces, J6 RATE, J7 Conn_02x13_Odd_Even, Q1 BSS806NE, Q2 BSS806NE, Q3 BSS806NE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

Commit message: CleanUp
Parts:
- removed J6: RATE, TestPoint:TestPoint_THTPad_D1.5mm_Drill0.7mm
- removed Q2: BSS806NE, Package_TO_SOT_SMD:SOT-23
- removed R11: 10k, Resistor_SMD:R_1206_3216Metric_Pad1.30x1.75mm_HandSolder
- added C21: 100n, Capacitor_SMD:C_1206_3216Metric_Pad1.33x1.80mm_HandSolder, B.Cu at (56.2, 103.4)
- added C23: 10u, Capacitor_SMD:C_1206_3216Metric_Pad1.33x1.80mm_HandSolder, B.Cu at (56.2, 105.9)
- added C25: 100n, Capacitor_SMD:C_1206_3216Metric_Pad1.33x1.80mm_HandSolder, B.Cu at (65.0, 93.2)
- added C29: 100n, Capacitor_SMD:C_1206_3216Metric_Pad1.33x1.80mm_HandSolder, B.Cu at (61.2, 97.0)
- added C30: 100n, Capacitor_SMD:C_1206_3216Metric_Pad1.33x1.80mm_HandSolder, B.Cu at (70.8, 109.1)
- added C31: 10u, Capacitor_SMD:C_1206_3216Metric_Pad1.33x1.80mm_HandSolder, B.Cu at (73.3, 109.1)
- added C32: 47u, Capacitor_SMD:C_1206_3216Metric_Pad1.33x1.80mm_HandSolder, B.Cu at (75.8, 109.1)
- added C33: 100n, Capacitor_SMD:C_1206_3216Metric_Pad1.33x1.80mm_HandSolder, B.Cu at (51.7, 87.5)
- added C34: 10u, Capacitor_SMD:C_1206_3216Metric_Pad1.33x1.80mm_HandSolder, B.Cu at (51.7, 90.0)
- added JP16: Jumper_3_Open, Jumper:SolderJumper-3_P1.3mm_Open_RoundedPad1.0x1.5mm, B.Cu at (68.2, 116.1)
- Q1: value BSS806NE -> MMBT4403L
- R2: value 470 -> 100
- R3: value 910 -> 100
- R4: value 10k -> 20k
- R5: value 10k -> 7k15
- R6, R7: value 220 -> 10k
- U3: footprint modules:hy711_module_smd -> Package_SO:SO-16_5.3x10.2mm_P1.27mm
- moved R8 59.4 mm to (103.8, 88.8)
- moved R3 36.2 mm to (61.9, 89.4), turned to 270 degrees
- moved R2 30.0 mm to (68.2, 89.4), turned to 270 degrees
- moved R6 28.7 mm to (79.0, 104.0), turned to 180 degrees
- moved R4 22.5 mm to (56.2, 100.8), turned to 0 degrees
- moved R5 17.7 mm to (56.2, 98.3), turned to 180 degrees
- moved C14 17.5 mm to (60.0, 109.1)
- moved Q1 15.9 mm to (60.6, 104.6), turned to 180 degrees
- moved C18 14.5 mm to (62.5, 109.1)
- moved C19 12.8 mm to (65.0, 109.1)
- moved R7 7.26 mm to (74.6, 97.0), turned to 270 degrees
- moved U3 5.85 mm to (67.6, 100.8), turned to 0 degrees
- moved TP4 4.44 mm to (99.3, 90.7)
Connections:
- C14 pad 1: +5VA -> Net-(C14-Pad1)
- C18 pad 1: +5VA -> Net-(C14-Pad1)
- C19 pad 1: +5VA -> Net-(C14-Pad1)
- J1 pad 1: Net-(J1-Pad1) -> Net-(C21-Pad1)
- J7 pad 10: (no net) -> Net-(J7-Pad10)
- J7 pad 2: (no net) -> Net-(J7-Pad2)
- J7 pad 3: (no net) -> Net-(J7-Pad3)
- J7 pad 5: (no net) -> Net-(J7-Pad5)
- J7 pad 7: (no net) -> Net-(J7-Pad7)
- J7 pad 9: (no net) -> Net-(J7-Pad9)
- Q1 pad 2: GND -> Net-(C14-Pad1)
- Q1 pad 3: Net-(Q1-Pad3) -> Net-(C21-Pad1)
- R2 pad 1: Net-(R2-Pad1) -> Net-(J4-Pad1)
- R2 pad 2: /DT -> Net-(C25-Pad1)
- R3 pad 1: /DT -> Net-(J3-Pad1)
- R3 pad 2: GND -> Net-(C25-Pad2)
- R4 pad 1: +5VA -> Net-(C21-Pad1)
- R4 pad 2: Net-(Q1-Pad3) -> Net-(R4-Pad2)
- R5 pad 1: Net-(Q1-Pad1) -> Net-(R4-Pad2)
- R6 pad 1: Net-(Q2-Pad1) -> GND
- R7 pad 1: Net-(Q1-Pad1) -> GND
- R8 pad 1: Net-(Q2-Pad1) -> GND
- R8 pad 2: GND -> /DT
- U2 pad 1: (no net) -> Net-(U2-Pad1)
- U2 pad 2: (no net) -> Net-(U2-Pad2)
- U2 pad 6: (no net) -> Net-(U2-Pad6)
- U2 pad 7: (no net) -> Net-(U2-Pad7)
- U2 pad 8: (no net) -> Net-(U2-Pad8)
- U3 pad 1: Net-(J1-Pad1) -> Net-(C14-Pad1)
- U3 pad 10: GND -> Net-(U3-Pad10)
- U3 pad 2: Net-(J2-Pad1) -> Net-(Q1-Pad1)
- U3 pad 3: Net-(J3-Pad1) -> Net-(C21-Pad1)
- U3 pad 4: Net-(J4-Pad1) -> Net-(R4-Pad2)
- U3 pad 5: (no net) -> GND
- U3 pad 6: (no net) -> Net-(C29-Pad1)
- U3 pad 7: +5VA -> Net-(C25-Pad1)
- U3 pad 8: Net-(Q1-Pad3) -> Net-(C25-Pad2)
- U3 pad 9: Net-(R2-Pad1) -> Net-(U3-Pad9)
Routing:
- net +3V3: track 18.3 -> 70.3 mm
- net Net-(R2-Pad1): track 49.4 -> 0.00 mm
- net GND: track 145.9 -> 183.6 mm, vias 95 -> 100
- net Net-(C21-Pad1): track 0.00 -> 31.8 mm
- net /RATE: track 73.9 -> 47.0 mm, vias 2 -> 0
- net /DT: track 18.0 -> 42.7 mm, vias 0 -> 2
- net Net-(Q1-Pad3): track 20.3 -> 0.00 mm
- net Net-(J2-Pad1): track 16.3 -> 0.00 mm
- net Net-(J1-Pad1): track 15.1 -> 0.00 mm
- net Net-(J6-Pad1): track 13.1 -> 0.00 mm
- net Net-(C14-Pad1): track 0.00 -> 10.4 mm
- net Net-(J4-Pad1): track 16.6 -> 6.52 mm
- net Net-(C25-Pad1): track 0.00 -> 9.31 mm
- net Net-(R4-Pad2): track 0.00 -> 9.22 mm
- net +5VA: track 56.9 -> 49.1 mm
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- added copper zone on B.Cu, net (none)
- added copper zone on F.Cu, net (none)
- added copper zone on B.Cu, net +3V3
- added copper zone on B.Cu, net Net-(C14-Pad1)
- added copper zone on B.Cu, net Net-(C21-Pad1)
Other:
- board text added: "5V"
- board text added: "FORCELOG_MOD HX711-A REV.C"
