File: pcb/pcb_motherboard_dev/pcb_motherboard_dev.kicad_pcb (KiCad board)
At the start: 4 copper layers, 100 x 100 mm, 176 parts, among them J1 Screw_Terminal_01x02, J13 LED, J2 Conn_01x04_Male, J4 Conn_02x04_Odd_Even, J5 AudioJack3, J6 SYNC, J7 Conn_02x13_Odd_Even, J8 Micro_SD_Card, Q1 DMG9926USD, Q2 IRF7410TRPBF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

Commit message: CleanUp
Connections:
- net /CONTROLLER/IO_5|V~CS renamed /CONTROLLER/IO_5|V~{CS}
- net /POWER/~LED_CHRG renamed /POWER/~{LED_CHRG}
- net /POWER/~LED_STBY renamed /POWER/~{LED_STBY}
Other:
- net class Default removed
