File: pcb/pcb_motherboard_dev/CONTROLLER.kicad_sch (KiCad schematic)
At the start: 44 parts, among them J7 Conn_02x13_Odd_Even, Q3 IRLML2244TRPBF, Q4 BSS806NE, SW3 SW_DIP_x01, U11 DS18B20Z, U12 2POS_JUMPER_8BIT, U7 74HC165, U8 ESP32-WROOM-32, Y1 32.768 kHz

Commit message: PCB MB-DEV update
+Added a jumper for GPIO12 for flashing and setting efuse for 3.3 Flash operation
+Added Text Variables to Schematic and PCB
+introduced versioning of pcb
+added filenames and version to schematic sheets
Parts:
- added TP23: FLASH, PinHeader:PinHeader_1x02_P2.54mm_Vertical, symbol Connector:TestPoint_2Pole
Connections:
- net HMISO: now also TP23.2; no longer U8.14 (IO12)
- new net: TP23.1, U8.14 (IO12)
Other:
- title: (none) -> ForcelogADC_MB-DEV_v${VERSION}
