File: pcb/pcb_motherboard_dev/POWER.kicad_sch (KiCad schematic)
At the start: 45 parts, among them J1 Screw_Terminal_01x02, J13 LED, J2 Conn_01x04_Male, Q1 DMG9926USD, Q2 IRF7410TRPBF, Q6 IRF7410TRPBF, SW2 SW_DIP_x01, U1 TP4056, U2 LP38501, U3 TP4056withprotect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

Commit message: PCB MB-DEV update
+Added a jumper for GPIO12 for flashing and setting efuse for 3.3 Flash operation
+Added Text Variables to Schematic and PCB
+introduced versioning of pcb
+added filenames and version to schematic sheets
Other:
- title: (none) -> ForcelogADC_MB-DEV_v${VERSION}
Changed lines of the file:
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@@
 (kicad_sch (version 20211123) (generator eeschema)
   (paper "A4")
+  (title_block
+    (title "ForcelogADC_MB-DEV_v${VERSION}")
+    (rev "${REVISION}")
+  )
   (junction (at 49.53 68.58) (diameter 0) (color 0 0 0 0)
   )
@@
     (pin "7")
     (pin "8")
+    (pin "3")
+    (pin "4")
+    (pin "5")
+    (pin "6")
   )
   (symbol (lib_id "Device:Q_Dual_NMOS_S1G1S2G2D2D2D1D1") (at 137.16 109.22 270) (unit 2)
@@
       (effects (font (size 1.27 1.27)) hide)
     )
+    (pin "1")
+    (pin "2")
+    (pin "7")
+    (pin "8")
     (pin "3")
     (pin "4")
