File: pcb/pcb_motherboard_dev/SD.kicad_sch (KiCad schematic)
At the start: 12 parts, among them J8 Micro_SD_Card

Commit message: PCB MB-DEV update
+Added a jumper for GPIO12 for flashing and setting efuse for 3.3 Flash operation
+Added Text Variables to Schematic and PCB
+introduced versioning of pcb
+added filenames and version to schematic sheets
Other:
- title: (none) -> ForcelogADC_MB-DEV_v${VERSION}
Changed lines of the file:
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@@
 (kicad_sch (version 20211123) (generator eeschema)
   (paper "A4")
+  (title_block
+    (title "ForcelogADC_MB-DEV_v${VERSION}")
+    (rev "${REVISION}")
+  )
   (junction (at 151.13 102.87) (diameter 0) (color 0 0 0 0)
   )
@@
     (pin "2")
   )
-  (symbol (lib_id "Device:C") (at 177.8 106.68 0)
+  (symbol (lib_id "Device:C") (at 177.8 106.68 0) (unit 1)
     (in_bom yes) (on_board yes)
     (property "Reference" "C11" (id 0) (at 180.721 105.5116 0)
@@
     (pin "2")
   )
-  (symbol (lib_id "Device:C") (at 167.64 106.68 0)
+  (symbol (lib_id "Device:C") (at 167.64 106.68 0) (unit 1)
     (in_bom yes) (on_board yes)
     (property "Reference" "C9" (id 0) (at 170.561 105.5116 0)
@@
     (pin "2")
   )
-  (symbol (lib_id "power:GND") (at 140.97 114.3 90) (mirror x)
+  (symbol (lib_id "power:GND") (at 140.97 114.3 90) (mirror x) (unit 1)
     (in_bom yes) (on_board yes)
     (property "Reference" "#PWR050" (id 0) (at 147.32 114.3 0)
@@
     (pin "1")
   )
-  (symbol (lib_id "Device:R") (at 137.16 114.3 270) (mirror x)
+  (symbol (lib_id "Device:R") (at 137.16 114.3 270) (mirror x) (unit 1)
     (in_bom yes) (on_board yes)
     (property "Reference" "R25" (id 0) (at 135.89 111.76 90)
@@
     (pin "2")
   )
-  (symbol (lib_id "power:+3.3V") (at 140.97 104.14 270) (mirror x)
+  (symbol (lib_id "power:+3.3V") (at 140.97 104.14 270) (mirror x) (unit 1)
     (in_bom yes) (on_board yes)
     (property "Reference" "#PWR047" (id 0) (at 137.16 104.14 0)
@@
     (pin "1")
   )
-  (symbol (lib_id "Device:R") (at 137.16 104.14 270) (mirror x)
+  (symbol (lib_id "Device:R") (at 137.16 104.14 270) (mirror x) (unit 1)
     (in_bom yes) (on_board yes)
     (property "Reference" "R23" (id 0) (at 135.89 101.6 90)
@@
     (pin "2")
   )
-  (symbol (lib_id "power:+3.3V") (at 140.97 121.92 270) (mirror x)
+  (symbol (lib_id "power:+3.3V") (at 140.97 121.92 270) (mirror x) (unit 1)
     (in_bom yes) (on_board yes)
     (property "Reference" "#PWR051" (id 0) (at 137.16 121.92 0)
@@
     (pin "1")
   )
-  (symbol (lib_id "Device:R") (at 137.16 121.92 270) (mirror x)
+  (symbol (lib_id "Device:R") (at 137.16 121.92 270) (mirror x) (unit 1)
     (in_bom yes) (on_board yes)
     (property "Reference" "R26" (id 0) (at 135.89 119.38 90)
@@
     (pin "2")
   )
-  (symbol (lib_id "power:GND") (at 165.1 111.76 0) (mirror y)
+  (symbol (lib_id "power:GND") (at 165.1 111.76 0) (mirror y) (unit 1)
     (in_bom yes) (on_board yes)
     (property "Reference" "#PWR067" (id 0) (at 165.1 118.11 0)
@@
     (pin "1")
   )
-  (symbol (lib_id "Device:C") (at 157.48 106.68 0)
+  (symbol (lib_id "Device:C") (at 157.48 106.68 0) (unit 1)
     (in_bom yes) (on_board yes)
     (property "Reference" "C8" (id 0) (at 160.401 105.5116 0)
@@
     (pin "2")
   )
-  (symbol (lib_id "power:+3.3V") (at 176.53 93.98 0) (mirror y)
+  (symbol (lib_id "power:+3.3V") (at 176.53 93.98 0) (mirror y) (unit 1)
     (in_bom yes) (on_board yes)
     (property "Reference" "#PWR073" (id 0) (at 176.53 97.79 0)
@@
     (pin "1")
   )
-  (symbol (lib_id "power:GND") (at 133.35 116.84 90) (mirror x)
+  (symbol (lib_id "power:GND") (at 133.35 116.84 90) (mirror x) (unit 1)
     (in_bom yes) (on_board yes)
     (property "Reference" "#PWR046" (id 0) (at 139.7 116.84 0)
@@
     (pin "1")
   )
-  (symbol (lib_id "power:+3.3V") (at 140.97 109.22 270) (mirror x)
+  (symbol (lib_id "power:+3.3V") (at 140.97 109.22 270) (mirror x) (unit 1)
     (in_bom yes) (on_board yes)
     (property "Reference" "#PWR048" (id 0) (at 137.16 109.22 0)
@@
     (pin "1")
   )
-  (symbol (lib_id "Device:R") (at 137.16 109.22 270) (mirror x)
+  (symbol (lib_id "Device:R") (at 137.16 109.22 270) (mirror x) (unit 1)
     (in_bom yes) (on_board yes)
     (property "Reference" "R24" (id 0) (at 135.89 106.68 90)
@@
     (pin "2")
   )
-  (symbol (lib_id "power:GND") (at 82.55 127 0) (mirror y)
+  (symbol (lib_id "power:GND") (at 82.55 127 0) (mirror y) (unit 1)
     (in_bom yes) (on_board yes)
     (property "Reference" "#PWR044" (id 0) (at 82.55 133.35 0)
@@
     (pin "1")
   )
-  (symbol (lib_id "Connector:Micro_SD_Card") (at 102.87 111.76 0) (mirror y)
+  (symbol (lib_id "Connector:Micro_SD_Card") (at 102.87 111.76 0) (mirror y) (unit 1)
     (in_bom yes) (on_board yes)
     (property "Reference" "J8" (id 0) (at 104.14 95.885 0))
@@
     (pin "9")
   )
-  (symbol (lib_id "Device:L") (at 160.02 93.98 90)
+  (symbol (lib_id "Device:L") (at 160.02 93.98 90) (unit 1)
     (in_bom yes) (on_board yes)
     (property "Reference" "L1" (id 0) (at 160.02 89.154 90))
@@
     (pin "2")
   )
-  (symbol (lib_id "Device:D_Schottky_Dual_Series_AKC") (at 151.13 93.98 90) (mirror x)
+  (symbol (lib_id "Device:D_Schottky_Dual_Series_AKC") (at 151.13 93.98 90) (mirror x) (unit 1)
     (in_bom yes) (on_board yes)
     (property "Reference" "D6" (id 0) (at 149.1234 93.98 90)
@@
     (pin "3")
   )
-  (symbol (lib_id "power:GND") (at 151.13 86.36 180)
+  (symbol (lib_id "power:GND") (at 151.13 86.36 180) (unit 1)
     (in_bom yes) (on_board yes)
     (property "Reference" "#PWR053" (id 0) (at 151.13 80.01 0)
@@
     (pin "1")
   )
-  (symbol (lib_id "Device:C") (at 187.96 106.68 0)
+  (symbol (lib_id "Device:C") (at 187.96 106.68 0) (unit 1)
     (in_bom yes) (on_board yes)
     (property "Reference" "C13" (id 0) (at 190.881 105.5116 0)
@@
     (pin "2")
   )
-  (symbol (lib_id "power:+3.3V") (at 156.21 133.35 0) (mirror y)
+  (symbol (lib_id "power:+3.3V") (at 156.21 133.35 0) (mirror y) (unit 1)
     (in_bom yes) (on_board yes)
     (property "Reference" "#PWR054" (id 0) (at 156.21 137.16 0)
@@
     (pin "1")
   )
-  (symbol (lib_id "power:GND") (at 156.21 135.89 0) (mirror y)
+  (symbol (lib_id "power:GND") (at 156.21 135.89 0) (mirror y) (unit 1)
     (in_bom yes) (on_board yes)
     (property "Reference" "#PWR066" (id 0) (at 156.21 142.24 0)
