File: pcb/pcb_motherboard_dev/connectors.kicad_sch (KiCad schematic)
At the start: 27 parts, among them J5 AudioJack3, J6 SYNC, Q5 BSS806NE, Q7 BSS806NE, SW1 SW_Push, U13 DS18B20Z, U5 EL357NC, U6 EL357NC

Commit message: PCB MB-DEV update
+Added a jumper for GPIO12 for flashing and setting efuse for 3.3 Flash operation
+Added Text Variables to Schematic and PCB
+introduced versioning of pcb
+added filenames and version to schematic sheets
Other:
- title: (none) -> ForcelogADC_MB-DEV_v${VERSION}
