File: pcb/pcb_motherboard_dev/ft232.kicad_sch (KiCad schematic)
At the start: 7 parts, among them U10 FT232breakout

Commit message: PCB MB-DEV update
+Added a jumper for GPIO12 for flashing and setting efuse for 3.3 Flash operation
+Added Text Variables to Schematic and PCB
+introduced versioning of pcb
+added filenames and version to schematic sheets
Other:
- title: (none) -> ForcelogADC_MB-DEV_v${VERSION}
Changed lines of the file:
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@@
 (kicad_sch (version 20211123) (generator eeschema)
   (paper "A4")
+  (title_block
+    (title "ForcelogADC_MB-DEV_v${VERSION}")
+    (rev "${REVISION}")
+  )
   (junction (at 190.5 97.79) (diameter 0) (color 0 0 0 0)
   )
@@
     (effects (font (size 1.27 1.27)) (justify right))
   )
-  (symbol (lib_id "Device:R") (at 119.38 110.49 270)
+  (symbol (lib_id "Device:R") (at 119.38 110.49 270) (unit 1)
     (in_bom yes) (on_board yes)
     (property "Reference" "R19" (id 0) (at 119.38 107.95 90))
@@
     (pin "2")
   )
-  (symbol (lib_id "power:+3.3V") (at 106.68 102.87 0) (mirror y)
+  (symbol (lib_id "power:+3.3V") (at 106.68 102.87 0) (mirror y) (unit 1)
     (in_bom yes) (on_board yes)
     (property "Reference" "#PWR096" (id 0) (at 106.68 106.68 0)
@@
     (pin "1")
   )
-  (symbol (lib_id "power:GND") (at 106.68 118.11 0)
+  (symbol (lib_id "power:GND") (at 106.68 118.11 0) (unit 1)
     (in_bom yes) (on_board yes)
     (property "Reference" "#PWR097" (id 0) (at 106.68 124.46 0)
@@
     (pin "1")
   )
-  (symbol (lib_id "Device:R") (at 146.05 99.06 270)
+  (symbol (lib_id "Device:R") (at 146.05 99.06 270) (unit 1)
     (in_bom yes) (on_board yes)
     (property "Reference" "R18" (id 0) (at 146.05 96.52 90))
@@
     (pin "2")
   )
-  (symbol (lib_id "power:+3.3V") (at 133.35 91.44 0) (mirror y)
+  (symbol (lib_id "power:+3.3V") (at 133.35 91.44 0) (mirror y) (unit 1)
     (in_bom yes) (on_board yes)
     (property "Reference" "#PWR098" (id 0) (at 133.35 95.25 0)
@@
     (pin "1")
   )
-  (symbol (lib_id "power:GND") (at 133.35 106.68 0)
+  (symbol (lib_id "power:GND") (at 133.35 106.68 0) (unit 1)
     (in_bom yes) (on_board yes)
     (property "Reference" "#PWR099" (id 0) (at 133.35 113.03 0)
@@
     (pin "1")
   )
-  (symbol (lib_id "Device:R") (at 152.4 102.87 270)
+  (symbol (lib_id "Device:R") (at 152.4 102.87 270) (unit 1)
     (in_bom yes) (on_board yes)
     (property "Reference" "R11" (id 0) (at 152.4 100.33 90))
@@
     (pin "2")
   )
-  (symbol (lib_id "Device:D_Schottky_Dual_Series_AKC") (at 133.35 99.06 90)
+  (symbol (lib_id "Device:D_Schottky_Dual_Series_AKC") (at 133.35 99.06 90) (unit 1)
     (in_bom yes) (on_board yes)
     (property "Reference" "D4" (id 0) (at 131.318 99.06 90)
@@
     (pin "3")
   )
-  (symbol (lib_id "Device:D_Schottky_Dual_Series_AKC") (at 106.68 110.49 90)
+  (symbol (lib_id "Device:D_Schottky_Dual_Series_AKC") (at 106.68 110.49 90) (unit 1)
     (in_bom yes) (on_board yes)
     (property "Reference" "D5" (id 0) (at 104.648 110.49 90)
@@
     (pin "3")
   )
-  (symbol (lib_id "modules:FT232breakout") (at 168.91 109.22 0)
+  (symbol (lib_id "modules:FT232breakout") (at 168.91 109.22 0) (unit 1)
     (in_bom yes) (on_board yes)
     (property "Reference" "U10" (id 0) (at 168.275 83.439 0))
@@
     (pin "9")
   )
-  (symbol (lib_id "power:+3.3V") (at 194.31 97.79 270)
+  (symbol (lib_id "power:+3.3V") (at 194.31 97.79 270) (unit 1)
     (in_bom yes) (on_board yes)
     (property "Reference" "#PWR0108" (id 0) (at 190.5 97.79 0)
@@
     (pin "1")
   )
-  (symbol (lib_id "power:+5VD") (at 179.07 93.98 270)
+  (symbol (lib_id "power:+5VD") (at 179.07 93.98 270) (unit 1)
     (in_bom yes) (on_board yes)
     (property "Reference" "#PWR0104" (id 0) (at 175.26 93.98 0)
@@
     (pin "1")
   )
-  (symbol (lib_id "power:GND") (at 179.07 105.41 90)
+  (symbol (lib_id "power:GND") (at 179.07 105.41 90) (unit 1)
     (in_bom yes) (on_board yes)
     (property "Reference" "#PWR0106" (id 0) (at 185.42 105.41 0)
@@
     (pin "1")
   )
-  (symbol (lib_id "power:GND") (at 179.07 101.6 90)
+  (symbol (lib_id "power:GND") (at 179.07 101.6 90) (unit 1)
     (in_bom yes) (on_board yes)
     (property "Reference" "#PWR0105" (id 0) (at 185.42 101.6 0)
@@
     (pin "1")
   )
-  (symbol (lib_id "power:GND") (at 138.43 138.43 0)
+  (symbol (lib_id "power:GND") (at 138.43 138.43 0) (unit 1)
     (in_bom yes) (on_board yes)
     (property "Reference" "#PWR0101" (id 0) (at 138.43 144.78 0)
@@
     (pin "1")
   )
-  (symbol (lib_id "power:+3.3V") (at 138.43 135.89 0) (mirror y)
+  (symbol (lib_id "power:+3.3V") (at 138.43 135.89 0) (mirror y) (unit 1)
     (in_bom yes) (on_board yes)
     (property "Reference" "#PWR0100" (id 0) (at 138.43 139.7 0)
@@
     (pin "2")
   )
-  (symbol (lib_id "power:GND") (at 190.5 105.41 0)
+  (symbol (lib_id "power:GND") (at 190.5 105.41 0) (unit 1)
     (in_bom yes) (on_board yes)
     (property "Reference" "#PWR0107" (id 0) (at 190.5 111.76 0)
@@
     (pin "1")
   )
-  (symbol (lib_id "power:+5VD") (at 138.43 149.86 270)
+  (symbol (lib_id "power:+5VD") (at 138.43 149.86 270) (unit 1)
     (in_bom yes) (on_board yes)
     (property "Reference" "#PWR0103" (id 0) (at 134.62 149.86 0)
