File: pcb/pcb_motherboard_dev/pcb_motherboard_dev.kicad_sch (KiCad schematic)
At the start: 8 parts

Commit message: PCB MB-DEV update
+Added a jumper for GPIO12 for flashing and setting efuse for 3.3 Flash operation
+Added Text Variables to Schematic and PCB
+introduced versioning of pcb
+added filenames and version to schematic sheets
Other:
- title: (none) -> ForcelogADC_MB-DEV_v${VERSION}
Changed lines of the file:
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@@
 (kicad_sch (version 20211123) (generator eeschema)
   (paper "A4")
+  (title_block
+    (title "ForcelogADC_MB-DEV_v${VERSION}")
+    (rev "${REVISION}")
+  )
   (no_connect (at 26.67 90.17))
   (no_connect (at 26.67 82.55))
@@
       (reference "TP22") (unit 1) (value "ID") (footprint "Connector_PinHeader_2.54mm:PinHeader_1x01_P2.54mm_Vertical")
     )
+    (path "/00000000-0000-0000-0000-00005fd1fa3f/5ea152c1-83db-4d14-9af9-99ab4f38f743"
+      (reference "TP23") (unit 1) (value "FLASH") (footprint "PinHeader:PinHeader_1x02_P2.54mm_Vertical")
+    )
     (path "/00000000-0000-0000-0000-00005fd1fa19/00000000-0000-0000-0000-00005fe127e5"
