File: pcb/pcb_motherboard_dev/sim_loadcell.kicad_sch (KiCad schematic)
At the start: 20 parts, among them J4 Conn_02x04_Odd_Even

Commit message: PCB MB-DEV update
+Added a jumper for GPIO12 for flashing and setting efuse for 3.3 Flash operation
+Added Text Variables to Schematic and PCB
+introduced versioning of pcb
+added filenames and version to schematic sheets
Other:
- title: (none) -> ForcelogADC_MB-DEV_v${VERSION}
Changed lines of the file:
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@@
 (kicad_sch (version 20211123) (generator eeschema)
   (paper "A4")
+  (title_block
+    (title "ForcelogADC_MB-DEV_v${VERSION}")
+    (rev "${REVISION}")
+  )
   (junction (at 181.61 95.25) (diameter 0) (color 0 0 0 0)
   )
@@
     (pin "2")
   )
-  (symbol (lib_id "Connector:TestPoint") (at 186.69 132.08 0)
+  (symbol (lib_id "Connector:TestPoint") (at 186.69 132.08 0) (unit 1)
     (in_bom yes) (on_board yes)
     (property "Reference" "TP14" (id 0) (at 188.1632 129.0828 0)
@@
     (pin "1")
   )
-  (symbol (lib_id "Connector:TestPoint") (at 194.31 132.08 0)
+  (symbol (lib_id "Connector:TestPoint") (at 194.31 132.08 0) (unit 1)
     (in_bom yes) (on_board yes)
     (property "Reference" "TP16" (id 0) (at 195.7832 129.0828 0)
@@
     (pin "1")
   )
-  (symbol (lib_id "Connector:TestPoint") (at 201.93 132.08 0)
+  (symbol (lib_id "Connector:TestPoint") (at 201.93 132.08 0) (unit 1)
     (in_bom yes) (on_board yes)
     (property "Reference" "TP18" (id 0) (at 203.4032 129.0828 0)
@@
     (pin "1")
   )
-  (symbol (lib_id "Connector:TestPoint") (at 209.55 132.08 0)
+  (symbol (lib_id "Connector:TestPoint") (at 209.55 132.08 0) (unit 1)
     (in_bom yes) (on_board yes)
     (property "Reference" "TP20" (id 0) (at 211.0232 129.0828 0)
@@
     (pin "1")
   )
-  (symbol (lib_id "Connector:TestPoint") (at 186.69 140.97 0)
+  (symbol (lib_id "Connector:TestPoint") (at 186.69 140.97 0) (unit 1)
     (in_bom yes) (on_board yes)
     (property "Reference" "TP15" (id 0) (at 188.1632 137.9728 0)
@@
     (pin "1")
   )
-  (symbol (lib_id "Connector:TestPoint") (at 194.31 140.97 0)
+  (symbol (lib_id "Connector:TestPoint") (at 194.31 140.97 0) (unit 1)
     (in_bom yes) (on_board yes)
     (property "Reference" "TP17" (id 0) (at 195.7832 137.9728 0)
@@
     (pin "1")
   )
-  (symbol (lib_id "Connector:TestPoint") (at 201.93 140.97 0)
+  (symbol (lib_id "Connector:TestPoint") (at 201.93 140.97 0) (unit 1)
     (in_bom yes) (on_board yes)
     (property "Reference" "TP19" (id 0) (at 203.4032 137.9728 0)
@@
     (pin "1")
   )
-  (symbol (lib_id "Connector:TestPoint") (at 209.55 140.97 0)
+  (symbol (lib_id "Connector:TestPoint") (at 209.55 140.97 0) (unit 1)
     (in_bom yes) (on_board yes)
     (property "Reference" "TP21" (id 0) (at 211.0232 137.9728 0)
