File: pcb/pcb_motherboard_module/pcb_motherboard_module.kicad_pcb (KiCad board)
At the start: 4 copper layers, 106.4 x 81.5 mm, 99 parts, among them J1 SW, J12 Conn_02x13_Odd_Even, J13 LED, J2 BAT, J3 POWER, J4 OWB, J5 COMM, J6 RGB, J7 SYNC, J8 Micro_SD_Card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

Commit message: CleanUp
Parts:
- removed J9: RFShield_TwoPieces, shields_rf:Shield_TE2118726-2
- removed JP2: Jumper_2_Open, Jumper:SolderJumper-2_P1.3mm_Open_TrianglePad1.0x1.5mm
- removed R22: 22k, Resistor_SMD:R_1206_3216Metric_Pad1.30x1.75mm_HandSolder
- added Q5: BSS806NE, Package_TO_SOT_SMD:SOT-23_Handsoldering, F.Cu at (178.4, 61.8)
- added R41: 100, Resistor_SMD:R_1206_3216Metric_Pad1.30x1.75mm_HandSolder, F.Cu at (168.9, 67.6)
- added R42: 10k, Resistor_SMD:R_1206_3216Metric_Pad1.30x1.75mm_HandSolder, F.Cu at (173.4, 82.2)
- added R43: 10k, Resistor_SMD:R_1206_3216Metric_Pad1.30x1.75mm_HandSolder, F.Cu at (170.8, 82.2)
- added R44: 10k, Resistor_SMD:R_1206_3216Metric_Pad1.30x1.75mm_HandSolder, F.Cu at (168.3, 82.2)
- added R45: 10k, Resistor_SMD:R_1206_3216Metric_Pad1.30x1.75mm_HandSolder, F.Cu at (165.7, 82.2)
- added R46: 10k, Resistor_SMD:R_1206_3216Metric_Pad1.30x1.75mm_HandSolder, F.Cu at (166.4, 99.3)
- added R47: 10k, Resistor_SMD:R_1206_3216Metric_Pad1.30x1.75mm_HandSolder, F.Cu at (168.9, 99.3)
- added R48: 10k, Resistor_SMD:R_1206_3216Metric_Pad1.30x1.75mm_HandSolder, F.Cu at (171.4, 99.3)
- added R49: 10k, Resistor_SMD:R_1206_3216Metric_Pad1.30x1.75mm_HandSolder, F.Cu at (174.0, 99.3)
- C18, C19: value C -> 25p
- R2: moved to B.Cu
- R21: value 100 -> 1k
- U2: footprint Package_TO_SOT_SMD:TO-252-5_TabPin6 -> Package_TO_SOT_SMD:TO-263-5_TabPin6
- moved R29 22.7 mm to (175.9, 82.2)
- moved R36 20.8 mm to (216.5, 105.7), turned to -90 degrees
- moved C12 16.5 mm to (165.7, 89.8), turned to -90 degrees
- moved R2 7.24 mm to (170.8, 122.8), turned to 0 degrees
- moved R13 5.08 mm to (156.2, 58.7)
- moved R15 5.08 mm to (151.1, 58.7)
- moved R11 4.45 mm to (184.8, 59.3)
- moved R24 3.42 mm to (214.0, 105.7)
- moved R25 3.42 mm to (211.5, 105.7)
- moved R34 3.42 mm to (209.5, 86.6)
- moved R23 3.42 mm to (219.1, 105.7)
- moved R26 3.42 mm to (208.9, 105.7)
- moved C11 3.42 mm to (215.9, 93.0)
- moved C9 3.42 mm to (212.7, 101.8)
- moved J8 3.42 mm to (214.0, 97.4)
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Connections:
- net /CONTROLLER/IO_5|V~CS renamed /CONTROLLER/IO_5|V~{CS}
- net /POWER/~LED_CHRG renamed /POWER/~{LED_CHRG}
- net /POWER/~LED_STBY renamed /POWER/~{LED_STBY}
- J8 pad 2: Net-(J8-Pad2) -> /CONTROLLER/HMSS
- R11 pad 1: Net-(J5-Pad2) -> Net-(J5-Pad3)
- R13 pad 1: Net-(J6-Pad4) -> Net-(J6-Pad2)
- R15 pad 1: Net-(J6-Pad2) -> Net-(J6-Pad4)
- R17 pad 1: Net-(R17-Pad1) -> Net-(J7-Pad6)
- R17 pad 2: Net-(J7-Pad6) -> Net-(R17-Pad2)
- R18 pad 1: Net-(J5-Pad3) -> Net-(J5-Pad2)
- R20 pad 1: /CONTROLLER/PING -> /CONTROLLER/SYNC
- R21 pad 1: GND -> Net-(Q5-Pad1)
- R21 pad 2: Net-(R21-Pad2) -> /CONTROLLER/SYNC
- R29 pad 2: Net-(JP2-Pad1) -> /CONTROLLER/BLUE
- R30 pad 1: Net-(R30-Pad1) -> /CONTROLLER/HMSS
- R34 pad 2: /CONTROLLER/PING -> /CONTROLLER/SYNC
- R36 pad 1: /CONTROLLER/DTR -> /CONTROLLER/HMSS
- U5 pad 1: Net-(R17-Pad1) -> Net-(R17-Pad2)
- U6 pad 1: /CONTROLLER/PING -> Net-(R41-Pad1)
- U6 pad 2: Net-(R21-Pad2) -> Net-(Q5-Pad3)
- U8 pad 12: /CONTROLLER/PING -> /CONTROLLER/SYNC
- U8 pad 25: Net-(R30-Pad1) -> /CONTROLLER/HMSS
Routing:
- net VDD: track 0.00 -> 133.1 mm
- net /CONTROLLER/DQ: track 2.16 -> 88.1 mm, vias 0 -> 3
- net /CONTROLLER/SYNC: track 0.00 -> 80.8 mm, vias 0 -> 3
- net /CONTROLLER/OWB_SENSE: track 18.6 -> 84.3 mm, vias 0 -> 1
- net /CONTROLLER/DTR: track 2.61 -> 61.8 mm, vias 0 -> 4
- net /CONTROLLER/HMSS: track 0.00 -> 42.0 mm, vias 0 -> 3
- net /CONTROLLER/RED: track 27.6 -> 68.6 mm, vias 1 -> 2
- net /CONTROLLER/CLK: track 0.00 -> 38.9 mm, vias 0 -> 2
- net /CONTROLLER/GREEN: track 15.9 -> 52.4 mm, vias 0 -> 1
- net /CONTROLLER/PING: track 34.9 -> 0.00 mm, vias 1 -> 0
- net GND: track 71.8 -> 104.4 mm, vias 52 -> 144
- net /CONTROLLER/BLUE: track 23.8 -> 53.7 mm
- net /CONTROLLER/TXD: track 2.41 -> 25.0 mm, vias 0 -> 1
- net /CONTROLLER/RXD: track 5.84 -> 24.9 mm, vias 0 -> 1
- net Net-(C11-Pad1): track 22.3 -> 6.14 mm, vias 2 -> 4
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- added copper zone on F.Cu, net GND
- added copper zone on B.Cu, net Net-(C11-Pad1)
- removed copper zone on F.Cu, net +3V3
Other:
- net class Default removed
- board text added: "BATMAN"
- board text added: "CC:BY-SA KPNBG.DE"
- board text added: "FORCELOG_ADC"
- board text added: "ID"
- board text added: "JLCJLCJLCJLC"
- board text added: "LDO"
- board text added: "M3"
- board text added: "M4"
- board text added: "MB_PROD"
- board text added: "REV.A"
- board text added: "SD"
